File: uC.kicad_sch (KiCad schematic)
At the start: 21 parts, among them J7 Conn_01x03, P12 Conn_02x10_Odd_Even, SW1 SW_Push, SW2 SW_Push, U1 RPi-Pico

Commit message: Comienza ruteo en pcb
Parts:
- D17: value LedRed -> SPI_ERR
- J7: value Conn_01x03 -> 1W
- SW1: value SW_Push -> PICO-RST; footprint Button_Switch_SMD:SW_Push_1P1T_NO_CK_KSC7xxJ -> Button_Switch_THT:SW_PUSH_6mm
- SW2: footprint Button_Switch_SMD:SW_Push_1P1T_NO_CK_KSC7xxJ -> Button_Switch_THT:SW_PUSH_6mm
Other:
- moved on the sheet: J7
Changed lines of the file:
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@@
 	(wire
 		(pts
-			(xy 115.57 41.91) (xy 109.22 41.91)
+			(xy 115.57 41.91) (xy 106.68 41.91)
 		)
 		(stroke
@@
 	(wire
 		(pts
-			(xy 109.22 39.37) (xy 110.49 39.37)
+			(xy 106.68 39.37) (xy 110.49 39.37)
 		)
 		(stroke
@@
 	(wire
 		(pts
-			(xy 109.22 44.45) (xy 110.49 44.45)
+			(xy 106.68 44.45) (xy 110.49 44.45)
 		)
 		(stroke
@@
 			)
 		)
-		(property "Value" "LedRed"
+		(property "Value" "SPI_ERR"
 			(at 175.26 213.36 90)
 			(effects
@@
 	(symbol
 		(lib_id "Connector_Generic:Conn_01x03")
-		(at 104.14 41.91 0)
+		(at 101.6 41.91 0)
 		(mirror y)
 		(unit 1)
@@
 		(dnp no)
 		(property "Reference" "J7"
-			(at 105.41 35.56 0)
+			(at 102.87 34.29 0)
 			(effects
 				(font
@@
 			)
 		)
-		(property "Value" "Conn_01x03"
-			(at 110.109 33.401 0)
+		(property "Value" "1W"
+			(at 102.87 36.83 0)
 			(effects
 				(font
@@
 				)
 				(justify left)
-				(hide yes)
 			)
 		)
 		(property "Footprint" "Connector_PinHeader_2.54mm:PinHeader_1x03_P2.54mm_Vertical"
-			(at 104.14 41.91 0)
+			(at 101.6 41.91 0)
 			(effects
 				(font
@@
 		)
 		(property "Datasheet" "~"
-			(at 104.14 41.91 0)
+			(at 101.6 41.91 0)
 			(effects
 				(font
@@
 		)
 		(property "Description" ""
-			(at 104.14 41.91 0)
+			(at 101.6 41.91 0)
 			(effects
 				(font
@@
 			)
 		)
-		(property "Footprint" "Button_Switch_SMD:SW_Push_1P1T_NO_CK_KSC7xxJ"
+		(property "Footprint" "Button_Switch_THT:SW_PUSH_6mm"
 			(at 95.25 52.07 0)
 			(effects
@@
 		(dnp no)
 		(property "Reference" "SW1"
-			(at 172.72 115.57 0)
+			(at 172.72 114.3 0)
 			(effects
 				(font
@@
 			)
 		)
-		(property "Value" "SW_Push"
-			(at 172.72 115.57 0)
+		(property "Value" "PICO-RST"
+			(at 172.72 116.84 0)
 			(effects
 				(font
 					(size 1.27 1.27)
 				)
-				(hide yes)
 			)
 		)
-		(property "Footprint" "Button_Switch_SMD:SW_Push_1P1T_NO_CK_KSC7xxJ"
+		(property "Footprint" "Button_Switch_THT:SW_PUSH_6mm"
 			(at 172.72 115.57 0)
 			(effects

Commit message: PCB: Faltan rutear 4 líneas de la capa bottom
Parts:
- JP1, JP2, JP3, JP4, JP5, JP6, JP7, JP8: footprint Connector_PinHeader_1.00mm:PinHeader_1x03_P1.00mm_Vertical_SMD_Pin1Left -> Connector_PinSocket_2.54mm:PinSocket_1x03_P2.54mm_Vertical
- R1: footprint Resistor_SMD:R_1206_3216Metric -> Resistor_THT:R_Axial_DIN0207_L6.3mm_D2.5mm_P7.62mm_Horizontal
Changed lines of the file:
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@@
 			)
 		)
-		(property "Footprint" "Connector_PinHeader_1.00mm:PinHeader_1x03_P1.00mm_Vertical_SMD_Pin1Left"
+		(property "Footprint" "Connector_PinSocket_2.54mm:PinSocket_1x03_P2.54mm_Vertical"
 			(at 38.1 106.68 0)
 			(effects
@@
 			)
 		)
-		(property "Footprint" "Connector_PinHeader_1.00mm:PinHeader_1x03_P1.00mm_Vertical_SMD_Pin1Left"
+		(property "Footprint" "Connector_PinSocket_2.54mm:PinSocket_1x03_P2.54mm_Vertical"
 			(at 38.1 123.19 0)
 			(effects
@@
 			)
 		)
-		(property "Footprint" "Connector_PinHeader_1.00mm:PinHeader_1x03_P1.00mm_Vertical_SMD_Pin1Left"
+		(property "Footprint" "Connector_PinSocket_2.54mm:PinSocket_1x03_P2.54mm_Vertical"
 			(at 62.23 102.87 0)
 			(effects
@@
 			)
 		)
-		(property "Footprint" "Connector_PinHeader_1.00mm:PinHeader_1x03_P1.00mm_Vertical_SMD_Pin1Left"
+		(property "Footprint" "Connector_PinSocket_2.54mm:PinSocket_1x03_P2.54mm_Vertical"
 			(at 62.23 135.89 0)
 			(effects
@@
 			)
 		)
-		(property "Footprint" "Connector_PinHeader_1.00mm:PinHeader_1x03_P1.00mm_Vertical_SMD_Pin1Left"
+		(property "Footprint" "Connector_PinSocket_2.54mm:PinSocket_1x03_P2.54mm_Vertical"
 			(at 38.1 90.17 0)
 			(effects
@@
 			)
 		)
-		(property "Footprint" "Connector_PinHeader_1.00mm:PinHeader_1x03_P1.00mm_Vertical_SMD_Pin1Left"
+		(property "Footprint" "Connector_PinSocket_2.54mm:PinSocket_1x03_P2.54mm_Vertical"
 			(at 62.23 152.4 0)
 			(effects
@@
 			)
 		)
-		(property "Footprint" "Connector_PinHeader_1.00mm:PinHeader_1x03_P1.00mm_Vertical_SMD_Pin1Left"
+		(property "Footprint" "Connector_PinSocket_2.54mm:PinSocket_1x03_P2.54mm_Vertical"
 			(at 38.1 139.7 0)
 			(effects
@@
 			)
 		)
-		(property "Footprint" "Connector_PinHeader_1.00mm:PinHeader_1x03_P1.00mm_Vertical_SMD_Pin1Left"
+		(property "Footprint" "Connector_PinSocket_2.54mm:PinSocket_1x03_P2.54mm_Vertical"
 			(at 62.23 119.38 0)
 			(effects
@@
 			)
 		)
-		(property "Footprint" "Resistor_SMD:R_1206_3216Metric"
+		(property "Footprint" "Resistor_THT:R_Axial_DIN0207_L6.3mm_D2.5mm_P7.62mm_Horizontal"
 			(at 117.348 36.83 90)
 			(effects
